File: Breadboard_PowerSupply.kicad_sch (KiCad schematic)
At the start: 0 parts

Commit message: Schematic Completed
Parts:
- added C1: 10u, Capacitor_THT:C_Disc_D3.0mm_W1.6mm_P2.50mm, symbol Device:C
- added C2: 0.1u, Capacitor_THT:C_Disc_D3.0mm_W1.6mm_P2.50mm, symbol Device:C
- added C3: 1u, Capacitor_THT:C_Disc_D3.0mm_W1.6mm_P2.50mm, symbol Device:C
- added D1: LED, LED_THT:LED_D5.0mm, symbol Device:LED
- added J1, J2: Conn_01x02_Pin, Connector_PinHeader_2.54mm:PinHeader_1x02_P2.54mm_Vertical, symbol Connector:Conn_01x02_Pin
- added J3, J4: Conn_01x03_Pin, Connector_PinHeader_2.54mm:PinHeader_1x03_P2.54mm_Vertical, symbol Connector:Conn_01x03_Pin
- added J5, J7: Screw_Terminal_01x02, TerminalBlock:TerminalBlock_bornier-2_P5.08mm, symbol Connector:Screw_Terminal_01x02
- added J6: Barrel_Jack_Switch, Connector_BarrelJack:BarrelJack_Horizontal, symbol Connector:Barrel_Jack_Switch
- added R1, R2: 330, Resistor_THT:R_Axial_DIN0204_L3.6mm_D1.6mm_P7.62mm_Horizontal, symbol Device:R
- added R3: 560, Resistor_THT:R_Axial_DIN0204_L3.6mm_D1.6mm_P7.62mm_Horizontal, symbol Device:R
- added S1: EG1218, digikey-footprints:Switch_Slide_11.6x4mm_EG1218, symbol dk_Slide-Switches:EG1218
- added U1: LM7805_TO220, Package_TO_SOT_THT:TO-220-3_Vertical, symbol Regulator_Linear:LM7805_TO220
- added U2: LM317_TO-220, Package_TO_SOT_THT:TO-220-3_Vertical, symbol Regulator_Linear:LM317_TO-220
Connections:
- new net: D1.2 (A), R2.1
- new net: R1.1, R3.2, U2.1 (ADJ)
- new net 12V: C1.1, R2.2, S1.1, U1.1 (VI), U2.3 (VI)
- new net 3.3V: C3.1, J3.1 (Pin_1), J4.1 (Pin_1), R1.2, U2.2 (VO)
- new net 5V: C2.1, J3.3 (Pin_3), J4.3 (Pin_3), U1.3 (VO)
- new net GND: C1.2, C2.2, C3.2, D1.1 (K), J1.1 (Pin_1), J2.1 (Pin_1), J5.1 (Pin_1), J6.2, J6.3, J7.1 (Pin_1), R3.1, U1.2 (GND)
- new net PWR_Input: J6.1, S1.2
- new net PWR_Output: J1.2 (Pin_2), J2.2 (Pin_2), J3.2 (Pin_2), J4.2 (Pin_2), J5.2 (Pin_2), J7.2 (Pin_2)
- no-connect marks 0 -> 1
Other:
- note added: "3.3V Circuit"
- note added: "Input and 5V Circuit"
- note added: "Output and Switches"
- title: (none) -> BreadBoard Power Supply
