File: schematic/Breadboard_PowerSupply.kicad_sch (KiCad schematic)
At the start: 17 parts, among them J1 Conn_01x02_Pin, J2 Conn_01x02_Pin, J3 Conn_01x03_Pin, J4 Conn_01x03_Pin, J5 Screw_Terminal_01x02, J6 Barrel_Jack_Switch, J7 Screw_Terminal_01x02, U1 LM7805_TO220, U2 LM317_TO-220

Commit message: Project Completed
Parts:
- D1: Purpose (none) -> Power input indicator
- J1, J2: Purpose (none) -> Output to the breadboard
- J3: Purpose (none) -> Output voltage selector 1
- J4: Purpose (none) -> Output voltage selector 2
- J5, J7: Purpose (none) -> Output to jumper wires
Connections:
- net PWR_Output renamed PWR_OUT_BOT
- net PWR_OUT_BOT: no longer J1.2 (Pin_2), J3.2 (Pin_2), J5.2 (Pin_2)
- new net PWR_OUT_TOP: J1.2 (Pin_2), J3.2 (Pin_2), J5.2 (Pin_2)
Other:
- moved on the sheet: D1, J5
Changed lines of the file:
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@@
 	(text "Output and Switches"
 		(exclude_from_sim no)
-		(at 159.512 30.226 0)
+		(at 159.512 29.21 0)
 		(effects
 			(font
@@
 	)
 	(junction
+		(at 93.98 130.81)
+		(diameter 0)
+		(color 0 0 0 0)
+	)
+	(junction
 		(at 50.8 100.33)
 		(diameter 0)
@@
 	)
 	(junction
-		(at 167.64 67.31)
-		(diameter 0)
-		(color 0 0 0 0)
-	)
-	(junction
 		(at 102.87 45.72)
 		(diameter 0)
@@
 	)
 	(junction
+		(at 167.64 68.58)
+		(diameter 0)
+		(color 0 0 0 0)
+	)
+	(junction
 		(at 93.98 113.03)
 		(diameter 0)
@@
 	(wire
 		(pts
-			(xy 93.98 129.54) (xy 93.98 134.62)
+			(xy 93.98 129.54) (xy 93.98 130.81)
 		)
 		(stroke
@@
 	(wire
 		(pts
-			(xy 167.64 58.42) (xy 167.64 67.31)
-		)
-		(stroke
-			(width 0)
-			(type default)
-		)
-	)
-	(wire
-		(pts
-			(xy 167.64 67.31) (xy 175.26 67.31)
+			(xy 167.64 68.58) (xy 175.26 68.58)
 		)
 		(stroke
@@
 	(wire
 		(pts
+			(xy 93.98 130.81) (xy 93.98 134.62)
+		)
+		(stroke
+			(width 0)
+			(type default)
+		)
+	)
+	(wire
+		(pts
 			(xy 58.42 95.25) (xy 58.42 100.33)
 		)
@@
 	(wire
 		(pts
-			(xy 167.64 73.66) (xy 167.64 67.31)
+			(xy 167.64 73.66) (xy 167.64 68.58)
 		)
 		(stroke
@@
 	(wire
 		(pts
-			(xy 50.8 129.54) (xy 58.42 129.54)
+			(xy 50.8 130.81) (xy 58.42 130.81)
 		)
 		(stroke
@@
 	(wire
 		(pts
-			(xy 170.18 64.77) (xy 175.26 64.77)
-		)
-		(stroke
-			(width 0)
-			(type default)
-		)
-	)
-	(wire
-		(pts
-			(xy 170.18 55.88) (xy 170.18 64.77)
+			(xy 170.18 66.04) (xy 175.26 66.04)
+		)
+		(stroke
+			(width 0)
+			(type default)
+		)
+	)
+	(wire
+		(pts
+			(xy 170.18 55.88) (xy 170.18 66.04)
 		)
 		(stroke
@@
 	(wire
 		(pts
+			(xy 168.91 95.25) (xy 168.91 109.22)
+		)
+		(stroke
+			(width 0)
+			(type default)
+		)
+	)
+	(wire
+		(pts
 			(xy 168.91 119.38) (xy 173.99 119.38)
 		)
@@
 	(wire
 		(pts
-			(xy 50.8 110.49) (xy 50.8 129.54)
+			(xy 50.8 110.49) (xy 50.8 130.81)
 		)
 		(stroke
@@
 	(wire
 		(pts
-			(xy 66.04 129.54) (xy 93.98 129.54)
-		)
-		(stroke
-			(width 0)
-			(type default)
-		)
-	)
-	(wire
-		(pts
-			(xy 168.91 95.25) (xy 168.91 109.22)
+			(xy 66.04 130.81) (xy 93.98 130.81)
+		)
+		(stroke
+			(width 0)
+			(type default)
+		)
+	)
+	(wire
+		(pts
+			(xy 167.64 58.42) (xy 167.64 68.58)
 		)
 		(stroke
@@
 		)
 	)
+	(label "PWR_OUT_BOT"
+		(at 168.91 102.87 0)
+		(effects
+			(font
+				(size 1.27 1.27)
+			)
+			(justify left bottom)
+		)
+	)
 	(label "5V"
 		(at 173.99 92.71 180)
@@
 		)
 	)
-	(label "PWR_Output"
-		(at 168.91 104.14 0)
-		(effects
-			(font
-				(size 1.27 1.27)
-			)
-			(justify left bottom)
-		)
-	)
 	(label "3.3V"
 		(at 173.99 97.79 180)
@@
 		)
 	)
-	(label "PWR_Output"
-		(at 170.18 52.07 0)
-		(effects
-			(font
-				(size 1.27 1.27)
-			)
-			(justify left bottom)
-		)
-	)
 	(label "12V"
 		(at 36.83 100.33 0)
@@
 		)
 	)
+	(label "PWR_OUT_TOP"
+		(at 170.18 49.53 0)
+		(effects
+			(font
+				(size 1.27 1.27)
+			)
+			(justify left bottom)
+		)
+	)
 	(rule_area
 		(polyline
@@
 		(polyline
 			(pts
-				(xy 205.74 31.75) (xy 205.74 142.24) (xy 149.86 142.24) (xy 149.86 31.75) (xy 196.85 31.75)
+				(xy 205.74 30.48) (xy 205.74 140.97) (xy 149.86 140.97) (xy 149.86 30.48) (xy 196.85 30.48)
 			)
 			(stroke
@@
 		(on_board yes)
 		(dnp no)
-		(fields_autoplaced yes)
 		(property "Reference" "J1"
 			(at 181.61 55.8799 0)
@@
 				)
 				(hide yes)
+			)
+		)
+		(property "Purpose" "Output to the breadboard"
+			(at 182.626 53.086 0)
+			(effects
+				(font
+					(size 1.27 1.27)
+				)
 			)
 		)
@@
 	(symbol
 		(lib_id "Device:LED")
-		(at 62.23 129.54 180)
+		(at 62.23 130.81 180)
 		(unit 1)
 		(exclude_from_sim no)
@@
 		(on_board yes)
 		(dnp no)
-		(fields_autoplaced yes)
 		(property "Reference" "D1"
-			(at 63.8175 121.92 0)
+			(at 63.8175 123.19 0)
 			(effects
 				(font
@@
 		)
 		(property "Value" "LED"
-			(at 63.8175 124.46 0)
+			(at 63.8175 125.73 0)
 			(effects
 				(font
@@
 		)
 		(property "Footprint" "LED_THT:LED_D5.0mm"
-			(at 62.23 129.54 0)
+			(at 62.23 130.81 0)
 			(effects
 				(font
@@
 		)
 		(property "Datasheet" "~"
-			(at 62.23 129.54 0)
+			(at 62.23 130.81 0)
 			(effects
 				(font
@@
 		)
 		(property "Description" "Light emitting diode"
-			(at 62.23 129.54 0)
+			(at 62.23 130.81 0)
 			(effects
 				(font
@@
 		)
 		(property "Sim.Pins" "1=K 2=A"
-			(at 62.23 129.54 0)
-			(effects
-				(font
-					(size 1.27 1.27)
-				)
-				(hide yes)
+			(at 62.23 130.81 0)
+			(effects
+				(font
+					(size 1.27 1.27)
+				)
+				(hide yes)
+			)
+		)
+		(property "Purpose" "Power input indicator"
+			(at 62.23 134.112 0)
+			(do_not_autoplace yes)
+			(effects
+				(font
+					(size 1.27 1.27)
+				)
 			)
 		)
@@
 			)
 		)
+		(property "Purpose" "Output to jumper wires"
+			(at 179.07 125.73 0)
+			(effects
+				(font
+					(size 1.27 1.27)
+				)
+			)
+		)
 		(pin "1"
 		)
@@
 		(on_board yes)
 		(dnp no)
-		(fields_autoplaced yes)
 		(property "Reference" "J4"
-			(at 180.34 93.9799 0)
+			(at 180.34 92.7099 0)
 			(effects
 				(font
@@
 		)
 		(property "Value" "Conn_01x03_Pin"
-			(at 180.34 96.5199 0)
+			(at 180.34 95.2499 0)
 			(effects
 				(font
@@
 				)
 				(hide yes)
+			)
+		)
+		(property "Purpose" "Output voltage selector 2"
+			(at 179.07 88.138 0)
+			(effects
+				(font
+					(size 1.27 1.27)
+				)
 			)
 		)
@@
 	(symbol
 		(lib_id "Connector:Screw_Terminal_01x02")
-		(at 180.34 67.31 0)
+		(at 180.34 68.58 0)
 		(mirror x)
 		(unit 1)
@@
 		(dnp no)
 		(property "Reference" "J5"
-			(at 182.88 67.3101 0)
+			(at 182.88 68.5801 0)
 			(effects
 				(font
@@
 		)
 		(property "Value" "Screw_Terminal_01x02"
-			(at 182.88 64.7701 0)
+			(at 182.88 66.0401 0)
 			(effects
 				(font
@@
 		)
 		(property "Footprint" "TerminalBlock:TerminalBlock_bornier-2_P5.08mm"
-			(at 180.34 67.31 0)
+			(at 180.34 68.58 0)
 			(effects
 				(font
@@
 		)
 		(property "Datasheet" "~"
-			(at 180.34 67.31 0)
+			(at 180.34 68.58 0)
 			(effects
 				(font
@@
 		)
 		(property "Description" "Generic screw terminal, single row, 01x02, script generated (kicad-library-utils/schlib/autogen/connector/)"
-			(at 180.34 67.31 0)
-			(effects
-				(font
-					(size 1.27 1.27)
-				)
-				(hide yes)
+			(at 180.34 68.58 0)
+			(effects
+				(font
+					(size 1.27 1.27)
+				)
+				(hide yes)
+			)
+		)
+		(property "Purpose" "Output to jumper wires"
+			(at 180.34 72.898 0)
+			(effects
+				(font
+					(size 1.27 1.27)
+				)
 			)
 		)
@@
 		(on_board yes)
 		(dnp no)
-		(fields_autoplaced yes)
 		(property "Reference" "J2"
-			(at 180.34 109.2199 0)
+			(at 180.34 107.9499 0)
 			(effects
 				(font
@@
 		)
 		(property "Value" "Conn_01x02_Pin"
-			(at 180.34 111.7599 0)
+			(at 180.34 110.4899 0)
 			(effects
 				(font
@@
 				)
 				(hide yes)
+			)
+		)
+		(property "Purpose" "Output to the breadboard"
+			(at 168.91 105.41 0)
+			(effects
+				(font
+					(size 1.27 1.27)
+				)
+				(justify right)
 			)
 		)
@@
 			)
 		)
+		(property "Purpose" "Output voltage selector 1"
+			(at 180.34 32.258 0)
+			(effects
+				(font
+					(size 1.27 1.27)
+				)
+			)
+		)
